Commit message: Make so101 mountable: so_arm_module/so_arm_joints macros
Splits so101's links/joints/ros2_control-joints out into reusable macros
(so101.module.xacro), following the same module/urdf split lekiwi_description
already uses for its own mountable base. so_arm_module takes a parent link
and mounts the arm via a fixed joint; "base_link" is renamed "arm_base_link"
so it can't collide with a host robot's own base_link. so_arm_joints exposes
just the <ros2_control> <joint> entries (no <hardware>/<plugin>), since the
STS bus can only have one plugin instance - a host with a shared bus (e.g. a
LeKiwi base) is meant to call it directly inside its own merged
<ros2_control> block instead of standing up a second one.

Also renames three properties (max_velocity_steps, max_velocity_rads,
max_torque_nm -> arm_-prefixed) that collided by name with unrelated
properties of the same names in lekiwi_description's base.control.xacro;
xacro properties share one flat namespace across included files, so the
collision would have silently handed one robot's velocity/torque limits to
the other once both were composed together.

so101.urdf.xacro keeps producing the exact same standalone robot as before,
now built by calling the new macros with parent="base_footprint" - verified
with a local xacro expansion (no ROS2 needed for macro-level xacro checks)
that link names, ros2_control joint count, and the max_velocity value are
unchanged from the pre-refactor output.

Co-Authored-By: Claude Sonnet 5 <noreply@anthropic.com>

File: so_arm_description/urdf/so101/so101.control.xacro (robot description, xacro)
@@ -18,8 +18,10 @@
        STS models could share this bus) -->
   <xacro:property name="sts_protocol_max_vel_steps" value="65535"/>  <!-- protocol's own u16 ceiling - let servo firmware, not us, set the real cap -->
-  <!-- Maximum allowable torque/velocity for each motor -->
-  <xacro:property name="max_velocity_steps" value="${sts_protocol_max_vel_steps}"/>  <!-- full hardware max -->
-  <xacro:property name="max_velocity_rads" value="${max_velocity_steps*2*pi/4096}"/>  <!-- rad/s -->
-  <xacro:property name="max_torque_nm" value="2.942"/>  <!-- N⋅m (30 kgf⋅cm for STS3215) -->
+  <!-- Maximum allowable torque/velocity for each motor. "arm_"-prefixed to avoid clashing
+       with lekiwi_description's own same-named properties (xacro's flat namespace) once
+       both are composed in base_so101. -->
+  <xacro:property name="arm_max_velocity_steps" value="${sts_protocol_max_vel_steps}"/>  <!-- full hardware max -->
+  <xacro:property name="arm_max_velocity_rads" value="${arm_max_velocity_steps*2*pi/4096}"/>  <!-- rad/s -->
+  <xacro:property name="arm_max_torque_nm" value="2.942"/>  <!-- N⋅m (30 kgf⋅cm for STS3215) -->
   <!-- Position-mode (Mode 0) internal servo PID, written to EEPROM on activate -->
   <xacro:property name="shoulder_pan_p_coefficient" value="14"/>

File: so_arm_description/urdf/so101/so101.urdf.xacro (robot description, xacro)
@@ -3,4 +3,5 @@
   <xacro:include filename="$(find so_arm_description)/urdf/so101/so101.common.xacro"/>
   <xacro:include filename="$(find so_arm_description)/urdf/so101/so101.control.xacro"/>
+  <xacro:include filename="$(find so_arm_description)/urdf/so101/so101.module.xacro"/>
   <!-- Arguments (externally settable, default to property values in so101.control.xacro) -->
   <xacro:arg name="serial_port"    default="${serial_port}"/>
@@ -42,435 +43,10 @@
   <!-- false = omit the wrist camera mount/body/frame links and their fixed joints below -->
   <xacro:arg name="wrist_camera_urdf" default="true"/>
-  <material name="light_grey">
-    <color rgba="${light_grey_rgba}"/>
-  </material>
-  <material name="charcoal">
-    <color rgba="${charcoal_rgba}"/>
-  </material>
-  <!-- LINKS -->
-  <!-- Dummy root link (KDL does not support inertia on root link) -->
+  <!-- Standalone robot, built from so101.module.xacro's macros. A host robot (base_so101)
+       calls so_arm_module/so_arm_joints directly instead of this block. -->
   <link name="base_footprint"/>
-  <joint name="world_to_base" type="fixed">
-    <parent link="base_footprint"/>
-    <child link="base_link"/>
+  <xacro:so_arm_module parent="base_footprint">
     <origin xyz="0 0 0" rpy="0 0 0"/>
-  </joint>
-  <!-- Base link -->
-  <link name="base_link">
-    <inertial>
-      <origin xyz="0.0137179 -5.19711e-05 0.0334843" rpy="0 0 0"/>
-      <mass value="0.147"/>
-      <inertia ixx="0.000114686" ixy="-4.59787e-07" ixz="4.97151e-06" iyy="0.000136117" iyz="9.75275e-08" izz="0.000130364"/>
-    </inertial>
-    <visual>
-      <origin xyz="-0.00636471 -9.94414e-05 -0.0024" rpy="1.5708 -1.67685e-15 1.5708"/>
-      <geometry>
-        <mesh filename="package://so_arm_description/meshes/so101/base_motor_holder_so101_v1.stl"/>
-      </geometry>
-      <material name="light_grey"/>
-    </visual>
-    <collision>
-      <origin xyz="-0.00636471 -9.94414e-05 -0.0024" rpy="1.5708 -1.67685e-15 1.5708"/>
-      <geometry>
-        <mesh filename="package://so_arm_description/meshes/so101/base_motor_holder_so101_v1.stl"/>
-      </geometry>
-    </collision>
-    <visual>
-      <origin xyz="-0.00636471 -8.97657e-09 -0.0024" rpy="1.5708 -2.78073e-29 1.5708"/>
-      <geometry>
-        <mesh filename="package://so_arm_description/meshes/so101/base_so101_v2.stl"/>
-      </geometry>
-      <material name="light_grey"/>
-    </visual>
-    <collision>
-      <origin xyz="-0.00636471 -8.97657e-09 -0.0024" rpy="1.5708 -2.78073e-29 1.5708"/>
-      <geometry>
-        <mesh filename="package://so_arm_description/meshes/so101/base_so101_v2.stl"/>
-      </geometry>
-    </collision>
-    <visual>
-      <origin xyz="0.0263353 -8.97657e-09 0.0437" rpy="-8.21148e-16 7.84513e-18 1.249e-15"/>
-      <geometry>
-        <mesh filename="package://so_arm_description/meshes/so101/sts3215_03a_v1.stl"/>
-      </geometry>
-      <material name="charcoal"/>
-    </visual>
-    <collision>
-      <origin xyz="0.0263353 -8.97657e-09 0.0437" rpy="-8.21148e-16 7.84513e-18 1.249e-15"/>
-      <geometry>
-        <mesh filename="package://so_arm_description/meshes/so101/sts3215_03a_v1.stl"/>
-      </geometry>
-    </collision>
-    <visual>
-      <origin xyz="-0.0309827 -0.000199441 0.0474" rpy="1.5708 -1.35493e-14 1.5708"/>
-      <geometry>
-        <mesh filename="package://so_arm_description/meshes/so101/waveshare_mounting_plate_so101_v2.stl"/>
-      </geometry>
-      <material name="light_grey"/>
-    </visual>
-    <collision>
-      <origin xyz="-0.0309827 -0.000199441 0.0474" rpy="1.5708 -1.35493e-14 1.5708"/>
-      <geometry>
-        <mesh filename="package://so_arm_description/meshes/so101/waveshare_mounting_plate_so101_v2.stl"/>
-      </geometry>
-    </collision>
-  </link>
-  <!-- Shoulder link -->
-  <link name="shoulder_link">
-    <inertial>
-      <origin xyz="0.0307604 -1.66727e-05 0.0252713" rpy="0 0 0"/>
-      <mass value="0.100006"/>
-      <inertia ixx="8.3759e-05" ixy="-7.55525e-08" ixz="-1.16342e-06" iyy="8.10403e-05" iyz="-1.54663e-07" izz="2.39783e-05"/>
-    </inertial>
-    <visual>
-      <origin xyz="0.0303992 0.000422241 0.0417" rpy="1.5708 -1.5708 0"/>
-      <geometry>
-        <mesh filename="package://so_arm_description/meshes/so101/sts3215_03a_v1.stl"/>
-      </geometry>
-      <material name="charcoal"/>
-    </visual>
-    <collision>
-      <origin xyz="0.0303992 0.000422241 0.0417" rpy="1.5708 -1.5708 0"/>
-      <geometry>
-        <mesh filename="package://so_arm_description/meshes/so101/sts3215_03a_v1.stl"/>
-      </geometry>
-    </collision>
-    <visual>
-      <origin xyz="0.0675992 -0.000177759 -0.0158499" rpy="1.5708 1.5708 0"/>
-      <geometry>
-        <mesh filename="package://so_arm_description/meshes/so101/motor_holder_so101_base_v1.stl"/>
-      </geometry>
-      <material name="light_grey"/>
-    </visual>
-    <collision>
-      <origin xyz="0.0675992 -0.000177759 -0.0158499" rpy="1.5708 1.5708 0"/>
-      <geometry>
-        <mesh filename="package://so_arm_description/meshes/so101/motor_holder_so101_base_v1.stl"/>
-      </geometry>
-    </collision>
-    <visual>
-      <origin xyz="-0.0122008 2.22413e-05 -0.0464" rpy="1.5708 0 3.14159"/>
-      <geometry>
-        <mesh filename="package://so_arm_description/meshes/so101/rotation_pitch_so101_v1.stl"/>
-      </geometry>
-      <material name="light_grey"/>
-    </visual>
-    <collision>
-      <origin xyz="-0.0122008 2.22413e-05 -0.0464" rpy="1.5708 0 3.14159"/>
-      <geometry>
-        <mesh filename="package://so_arm_description/meshes/so101/rotation_pitch_so101_v1.stl"/>
-      </geometry>
-    </collision>
-  </link>
-  <!-- Upper arm link -->
-  <link name="upper_arm_link">
-    <inertial>
-      <origin xyz="-0.0898471 -0.00838224 0.0184089" rpy="0 0 0"/>
-      <mass value="0.103"/>
-      <inertia ixx="4.08002e-05" ixy="-1.97819e-05" ixz="-4.03016e-08" iyy="0.000147318" iyz="8.97326e-09" izz="0.000142487"/>
-    </inertial>
-    <visual>
-      <origin xyz="-0.11257 -0.0155 0.0187" rpy="-3.14159 -5.27356e-16 -1.5708"/>
-      <geometry>
-        <mesh filename="package://so_arm_description/meshes/so101/sts3215_03a_v1.stl"/>
-      </geometry>
-      <material name="charcoal"/>
-    </visual>
-    <collision>
-      <origin xyz="-0.11257 -0.0155 0.0187" rpy="-3.14159 -5.27356e-16 -1.5708"/>
-      <geometry>
-        <mesh filename="package://so_arm_description/meshes/so101/sts3215_03a_v1.stl"/>
-      </geometry>
-    </collision>
-    <visual>
-      <origin xyz="-0.065085 0.012 0.0182" rpy="3.14159 -0 -1.30911e-30"/>
-      <geometry>
-        <mesh filename="package://so_arm_description/meshes/so101/upper_arm_so101_v1.stl"/>
-      </geometry>
-      <material name="light_grey"/>
-    </visual>
-    <collision>
-      <origin xyz="-0.065085 0.012 0.0182" rpy="3.14159 -0 -1.30911e-30"/>
-      <geometry>
-        <mesh filename="package://so_arm_description/meshes/so101/upper_arm_so101_v1.stl"/>
-      </geometry>
-    </collision>
-  </link>
-  <!-- Lower arm link -->
-  <link name="lower_arm_link">
-    <inertial>
-      <origin xyz="-0.0980701 0.00324376 0.0182831" rpy="0 0 0"/>
-      <mass value="0.104"/>
-      <inertia ixx="2.87438e-05" ixy="7.41152e-06" ixz="1.26409e-06" iyy="0.000159844" iyz="-4.90188e-08" izz="0.00014529"/>
-    </inertial>
-    <visual>
-      <origin xyz="-0.0648499 -0.032 0.0182" rpy="3.14159 -0 6.67202e-31"/>
-      <geometry>
-        <mesh filename="package://so_arm_description/meshes/so101/under_arm_so101_v1.stl"/>
-      </geometry>
-      <material name="light_grey"/>
-    </visual>
-    <collision>
-      <origin xyz="-0.0648499 -0.032 0.0182" rpy="3.14159 -0 6.67202e-31"/>
-      <geometry>
-        <mesh filename="package://so_arm_description/meshes/so101/under_arm_so101_v1.stl"/>
-      </geometry>
-    </collision>
-    <visual>
-      <origin xyz="-0.0648499 -0.032 0.018" rpy="-3.14159 -2.55351e-15 -1.83387e-30"/>
-      <geometry>
-        <mesh filename="package://so_arm_description/meshes/so101/motor_holder_so101_wrist_v1.stl"/>
-      </geometry>
-      <material name="light_grey"/>
-    </visual>
-    <collision>
-      <origin xyz="-0.0648499 -0.032 0.018" rpy="-3.14159 -2.55351e-15 -1.83387e-30"/>
-      <geometry>
-        <mesh filename="package://so_arm_description/meshes/so101/motor_holder_so101_wrist_v1.stl"/>
-      </geometry>
-    </collision>
-    <visual>
-      <origin xyz="-0.1224 0.0052 0.0187" rpy="-3.14159 -7.88861e-31 -3.14159"/>
-      <geometry>
-        <mesh filename="package://so_arm_description/meshes/so101/sts3215_03a_v1.stl"/>
-      </geometry>
-      <material name="charcoal"/>
-    </visual>
-    <collision>
-      <origin xyz="-0.1224 0.0052 0.0187" rpy="-3.14159 -7.88861e-31 -3.14159"/>
-      <geometry>
-        <mesh filename="package://so_arm_description/meshes/so101/sts3215_03a_v1.stl"/>
-      </geometry>
-    </collision>
-  </link>
-  <!-- Wrist link -->
-  <link name="wrist_link">
-    <inertial>
-      <origin xyz="-0.000103312 -0.0386143 0.0281156" rpy="0 0 0"/>
-      <mass value="0.079"/>
-      <inertia ixx="3.68263e-05" ixy="1.7893e-08" ixz="-5.28128e-08" iyy="2.5391e-05" iyz="3.6412e-06" izz="2.1e-05"/>
-    </inertial>
-    <visual>
-      <origin xyz="8.32667e-17 -0.0424 0.0306" rpy="1.5708 1.5708 0"/>
-      <geometry>
-        <mesh filename="package://so_arm_description/meshes/so101/sts3215_03a_no_horn_v1.stl"/>
-      </geometry>
-      <material name="charcoal"/>
-    </visual>
-    <collision>
-      <origin xyz="8.32667e-17 -0.0424 0.0306" rpy="1.5708 1.5708 0"/>
-      <geometry>
-        <mesh filename="package://so_arm_description/meshes/so101/sts3215_03a_no_horn_v1.stl"/>
-      </geometry>
-    </collision>
-    <visual>
-      <origin xyz="0 -0.028 0.0181" rpy="-1.5708 -1.5708 0"/>
-      <geometry>
-        <mesh filename="package://so_arm_description/meshes/so101/wrist_roll_pitch_so101_v2.stl"/>
-      </geometry>
-      <material name="light_grey"/>
-    </visual>
-    <collision>
-      <origin xyz="0 -0.028 0.0181" rpy="-1.5708 -1.5708 0"/>
-      <geometry>
-        <mesh filename="package://so_arm_description/meshes/so101/wrist_roll_pitch_so101_v2.stl"/>
-      </geometry>
-    </collision>
-  </link>
-  <!-- Gripper link -->
-  <link name="gripper_link">
-    <inertial>
-      <origin xyz="0.000213627 0.000245138 -0.025187" rpy="0 0 0"/>
-      <mass value="0.087"/>
-      <inertia ixx="2.75087e-05" ixy="-3.35241e-07" ixz="-5.7352e-06" iyy="4.33657e-05" iyz="-5.17847e-08" izz="3.45059e-05"/>
-    </inertial>
-    <visual>
-      <origin xyz="0.0077 0.0001 -0.0234" rpy="-1.5708 -5.19179e-17 -1.66533e-16"/>
-      <geometry>
-        <mesh filename="package://so_arm_description/meshes/so101/sts3215_03a_v1.stl"/>
-      </geometry>
-      <material name="charcoal"/>
-    </visual>
-    <collision>
-      <origin xyz="0.0077 0.0001 -0.0234" rpy="-1.5708 -5.19179e-17 -1.66533e-16"/>
-      <geometry>
-        <mesh filename="package://so_arm_description/meshes/so101/sts3215_03a_v1.stl"/>
-      </geometry>
-    </collision>
-    <visual>
-      <origin xyz="8.32667e-17 -0.000218214 0.000949706" rpy="-3.14159 -5.55112e-17 0"/>
-      <geometry>
-        <mesh filename="package://so_arm_description/meshes/so101/wrist_roll_follower_so101_v1.stl"/>
-      </geometry>
-      <material name="light_grey"/>
-    </visual>
-    <collision>
-      <origin xyz="8.32667e-17 -0.000218214 0.000949706" rpy="-3.14159 -5.55112e-17 0"/>
-      <geometry>
-        <mesh filename="package://so_arm_description/meshes/so101/wrist_roll_follower_so101_v1.stl"/>
-      </geometry>
-    </collision>
-  </link>
-  <!-- End effector frame (dummy link) -->
-  <link name="end_effector_link">
-    <inertial>
-      <origin xyz="0 0 0" rpy="0 0 0"/>
-      <mass value="1e-9"/>
-      <inertia ixx="0" ixy="0" ixz="0" iyy="0" iyz="0" izz="0"/>
-    </inertial>
-  </link>
-  <!-- SO-101 wrist camera mount (Hex-Nut Recess, 32x32 UVC module form factor). -->
-  <xacro:if value="${'$(arg wrist_camera_urdf)' == 'true'}">
-    <link name="wrist_camera_mount_link">
-      <inertial>
-        <origin xyz="0 0 0" rpy="0 0 0"/>
-        <mass value="0.02"/>
-        <inertia ixx="1e-5" ixy="0" ixz="0" iyy="1e-5" iyz="0" izz="1e-5"/>
-      </inertial>
-      <visual>
-        <origin xyz="0 0 0" rpy="0 0 0"/>
-        <geometry>
-          <mesh filename="package://so_arm_description/meshes/so101/wrist_camera_mount_so101_v1.stl" scale="0.001 0.001 0.001"/>
-        </geometry>
-        <material name="light_grey"/>
-      </visual>
-      <collision>
-        <origin xyz="0 0 0" rpy="0 0 0"/>
-        <geometry>
-          <mesh filename="package://so_arm_description/meshes/so101/wrist_camera_mount_so101_v1.stl" scale="0.001 0.001 0.001"/>
-        </geometry>
-      </collision>
-    </link>
-    <link name="wrist_camera_body_link">
-      <inertial>
-        <origin xyz="0 0 0" rpy="0 0 0"/>
-        <mass value="0.015"/>
-        <inertia ixx="1e-5" ixy="0" ixz="0" iyy="1e-5" iyz="0" izz="1e-5"/>
-      </inertial>
-      <visual>
-        <origin xyz="0 0 0" rpy="0 0 0"/>
-        <geometry>
-          <mesh filename="package://so_arm_description/meshes/so101/wrist_camera_so101_v1.stl"/>
-        </geometry>
-        <material name="charcoal"/>
-      </visual>
-      <collision>
-        <origin xyz="0 0 0" rpy="0 0 0"/>
-        <geometry>
-          <mesh filename="package://so_arm_description/meshes/so101/wrist_camera_so101_v1.stl"/>
-        </geometry>
-      </collision>
-    </link>
-    <!-- Upstream-aligned wrist camera frame (+X forward, -Y right, +Z up). -->
-    <link name="wrist_camera_frame">
-      <inertial>
-        <origin xyz="0 0 0" rpy="0 0 0"/>
-        <mass value="1e-9"/>
-        <inertia ixx="0" ixy="0" ixz="0" iyy="0" iyz="0" izz="0"/>
-      </inertial>
-    </link>
-    <!-- REP-103 optical frame (+Z forward, +X right, +Y down). -->
-    <link name="wrist_camera_optical_frame">
-      <inertial>
-        <origin xyz="0 0 0" rpy="0 0 0"/>
-        <mass value="1e-9"/>
-        <inertia ixx="0" ixy="0" ixz="0" iyy="0" iyz="0" izz="0"/>
-      </inertial>
-    </link>
-  </xacro:if>
-  <!-- Moving jaw link -->
-  <link name="moving_jaw_link">
-    <inertial>
-      <origin xyz="-0.00157495 -0.0300244 0.0192755" rpy="0 0 0"/>
-      <mass value="0.012"/>
-      <inertia ixx="6.61427e-06" ixy="-3.19807e-07" ixz="-5.90717e-09" iyy="1.89032e-06" iyz="-1.09945e-07" izz="5.28738e-06"/>
-    </inertial>
-    <visual>
-      <origin xyz="-5.55112e-17 -5.55112e-17 0.0189" rpy="9.53145e-17 6.93889e-18 1.24077e-24"/>
-      <geometry>
-        <mesh filename="package://so_arm_description/meshes/so101/moving_jaw_so101_v1.stl"/>
-      </geometry>
-      <material name="light_grey"/>
-    </visual>
-    <collision>
-      <origin xyz="-5.55112e-17 -5.55112e-17 0.0189" rpy="9.53145e-17 6.93889e-18 1.24077e-24"/>
-      <geometry>
-        <mesh filename="package://so_arm_description/meshes/so101/moving_jaw_so101_v1.stl"/>
-      </geometry>
-    </collision>
-  </link>
-  <!-- JOINTS -->
-  <!-- velocity="1e6" (unreachable) disables JointSaturationLimiter's clipping - the real
-       ceiling comes from max_velocity in the <ros2_control> block below. -->
-  <joint name="shoulder_pan_joint" type="revolute">
-    <parent link="base_link"/>
-    <child link="shoulder_link"/>
-    <origin xyz="${shoulder_pan_xyz}"/>
-    <axis xyz="0 0 1"/>
-    <limit lower="${shoulder_pan_lower}" upper="${shoulder_pan_upper}" effort="${max_torque_nm}" velocity="1e6"/>
-  </joint>
-  <joint name="shoulder_lift_joint" type="revolute">
-    <parent link="shoulder_link"/>
-    <child link="upper_arm_link"/>
-    <origin xyz="${shoulder_lift_xyz}" rpy="${shoulder_lift_rpy}"/>
-    <axis xyz="0 0 -1"/>
-    <limit lower="${shoulder_lift_lower}" upper="${shoulder_lift_upper}" effort="${max_torque_nm}" velocity="1e6"/>
-  </joint>
-  <joint name="elbow_flex_joint" type="revolute">
-    <parent link="upper_arm_link"/>
-    <child link="lower_arm_link"/>
-    <origin xyz="${elbow_flex_xyz}" rpy="${elbow_flex_rpy}"/>
-    <axis xyz="0 0 -1"/>
-    <limit lower="${elbow_flex_lower}" upper="${elbow_flex_upper}" effort="${max_torque_nm}" velocity="1e6"/>
-  </joint>
-  <joint name="wrist_flex_joint" type="revolute">
-    <parent link="lower_arm_link"/>
-    <child link="wrist_link"/>
-    <origin xyz="${wrist_flex_xyz}" rpy="${wrist_flex_rpy}"/>
-    <axis xyz="0 0 -1"/>
-    <limit lower="${wrist_flex_lower}" upper="${wrist_flex_upper}" effort="${max_torque_nm}" velocity="1e6"/>
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